File: RS485_Modbus_Wing.sch (KiCad schematic (older format))
At the start: 13 parts, among them J1 Screw_Terminal_01x02, U1 VOS617A, U2 VOS617A, U3 MAX487E

Commit message: Last_Change_Sch
Parts:
- added J1: feather long, TerminalBlock:TerminalBlock_Altech_AK300-2_P5.00mm, symbol Connector_Generic:Conn_01x16
- added J2: feather short, Connector_PinHeader_2.54mm:PinHeader_1x12_P2.54mm_Vertical, symbol Connector_Generic:Conn_01x12
- C1: value C_Small -> 0.1uF; footprint (none) -> Capacitor_SMD:C_0603_1608Metric; manf# (none) -> 0603F104Z160CT
- J1: footprint (none) -> TerminalBlock:TerminalBlock_Altech_AK300-2_P5.00mm
- R1, R2, R5, R6: footprint (none) -> Resistor_SMD:R_0603_1608Metric_Pad1.05x0.95mm_HandSolder; manf# (none) -> RC0603JR-071K1L
- R11, R7, R9: footprint (none) -> Resistor_SMD:R_0805_2012Metric_Pad1.15x1.40mm_HandSolder; manf# (none) -> RS-05K472JT
- R8: footprint (none) -> Resistor_SMD:R_0603_1608Metric_Pad1.05x0.95mm_HandSolder; manf# (none) -> 0603SAJ0121T5E
- U1, U2: footprint (none) -> Package_SO:SO-4_4.4x2.3mm_P1.27mm; symbol Isolatorr:VOS617A -> RS485_Modbus_Wing-rescue:VOS617A-Isolatorr; manf# (none) -> VOS617A-8T
- U3: value MAX487E -> MAX13487E; footprint (none) -> Package_SO:SOIC-8_3.9x4.9mm_P1.27mm; manf# (none) -> MAX13488EESA+T
Connections:
- net +3V3: now also J1.15 (Pin_15)
- net GND: now also J1.13 (Pin_13)
- new net A0: J1.12 (Pin_12)
- new net A1: J1.11 (Pin_11)
- new net A2: J1.10 (Pin_10)
- new net A3: J1.9 (Pin_9)
- new net A4: J1.8 (Pin_8)
- new net A5: J1.7 (Pin_7)
- new net AREF: J1.14 (Pin_14)
- new net D0: J2.3 (Pin_3)
- new net D1: J2.4 (Pin_4)
- new net D2: J2.5 (Pin_5)
- new net D3: J2.6 (Pin_6)
- new net D4: J2.7 (Pin_7)
- new net D5: J2.8 (Pin_8)
- new net D6: J2.9 (Pin_9)
- new net EN: J2.11 (Pin_11)
- new net FREE: J1.1 (Pin_1)
- new net MISO: J1.4 (Pin_4)
- new net MOSI: J1.5 (Pin_5)
- new net RX: J1.3 (Pin_3)
- new net SCK: J1.6 (Pin_6)
- new net SCL: J2.2 (Pin_2)
- new net SDA: J2.1 (Pin_1)
- new net TX: J1.2 (Pin_2)
- new net VBAT: J2.12 (Pin_12)
- new net VUSB: J2.10 (Pin_10)
- new net ~RST: J1.16 (Pin_16)
Changed lines of the file:
@@
 P 4190 2670
 F 0 "U3" H 3900 3270 50  0000 C CNN
-F 1 "MAX487E" H 3920 3180 50  0000 C CNN
-F 2 "" H 4190 1970 50  0001 C CNN
-F 3 "https://datasheets.maximintegrated.com/en/ds/MAX1487E-MAX491E.pdf" H 4190 2720 50  0001 C CNN
+F 1 "MAX13487E" H 3920 3180 50  0000 C CNN
+F 2 "Package_SO:SOIC-8_3.9x4.9mm_P1.27mm" H 4190 1970 50  0001 C CNN
+F 3 "https://www.mouser.mx/ProductDetail/Maxim-Integrated/MAX13488EESA%2bT?qs=CDqwynd4ZNrf75a2RFzJTw%3D%3D" H 4190 2720 50  0001 C CNN
+F 4 "MAX13488EESA+T" H 4190 2670 50  0001 C CNN "manf#"
 	1    4190 2670
 	1    0    0    -1
 $EndComp
 $Comp
-L Isolatorr:VOS617A U1
+L RS485_Modbus_Wing-rescue:VOS617A-Isolatorr U1
 U 1 1 5F9C2337
 P 1950 2900
 F 0 "U1" H 1701 2483 50  0000 C CNN
 F 1 "VOS617A" H 1850 2934 50  0000 C CNN
-F 2 "" H 1950 2900 50  0001 C CNN
-F 3 "" H 1950 2900 50  0001 C CNN
+F 2 "Package_SO:SO-4_4.4x2.3mm_P1.27mm" H 1950 2900 50  0001 C CNN
+F 3 "https://www.mouser.mx/ProductDetail/Vishay-Semiconductors/VOS617A-8T?qs=W2ZGOs8rFANtTo7lrKJrQA%3D%3D" H 1950 2900 50  0001 C CNN
+F 4 "VOS617A-8T" H 1950 2900 50  0001 C CNN "manf#"
 	1    1950 2900
 	1    0    0    -1
 $EndComp
 $Comp
-L Isolatorr:VOS617A U2
+L RS485_Modbus_Wing-rescue:VOS617A-Isolatorr U2
 U 1 1 5F9C0BC7
 P 1350 1770
 F 0 "U2" H 1366 1785 50  0000 C CNN
 F 1 "VOS617A" H 1166 1349 50  0000 C CNN
-F 2 "" H 1350 1770 50  0001 C CNN
-F 3 "" H 1350 1770 50  0001 C CNN
+F 2 "Package_SO:SO-4_4.4x2.3mm_P1.27mm" H 1350 1770 50  0001 C CNN
+F 3 "https://www.mouser.mx/ProductDetail/Vishay-Semiconductors/VOS617A-8T?qs=W2ZGOs8rFANtTo7lrKJrQA%3D%3D" H 1350 1770 50  0001 C CNN
+F 4 "VOS617A-8T" H 1350 1770 50  0001 C CNN "manf#"
 	1    1350 1770
 	-1   0    0    -1
@@
 F 0 "R7" H 3281 2114 50  0000 R CNN
 F 1 "4.7K" H 3281 2205 50  0000 R CNN
-F 2 "" H 3340 2160 50  0001 C CNN
-F 3 "~" H 3340 2160 50  0001 C CNN
+F 2 "Resistor_SMD:R_0805_2012Metric_Pad1.15x1.40mm_HandSolder" H 3340 2160 50  0001 C CNN
+F 3 "https://lcsc.com/product-detail/Chip-Resistor-Surface-Mount_FH-Guangdong-Fenghua-Advanced-Tech-RS-05K472JT_C115310.html" H 3340 2160 50  0001 C CNN
+F 4 "RS-05K472JT" H 3340 2160 50  0001 C CNN "manf#"
 	1    3340 2160
 	-1   0    0    1
@@
 F 0 "R6" H 1811 1704 50  0000 R CNN
 F 1 "1K" H 1811 1795 50  0000 R CNN
-F 2 "" H 1870 1750 50  0001 C CNN
-F 3 "~" H 1870 1750 50  0001 C CNN
+F 2 "Resistor_SMD:R_0603_1608Metric_Pad1.05x0.95mm_HandSolder" H 1870 1750 50  0001 C CNN
+F 3 "https://lcsc.com/product-detail/Chip-Resistor-Surface-Mount_YAGEO-RC0603JR-071K1L_C246023.html" H 1870 1750 50  0001 C CNN
+F 4 "RC0603JR-071K1L" H 1870 1750 50  0001 C CNN "manf#"
 	1    1870 1750
 	-1   0    0    1
@@
 F 0 "R2" H 820 1670 50  0000 L CNN
 F 1 "1K" H 810 1600 50  0000 L CNN
-F 2 "" H 970 1640 50  0001 C CNN
-F 3 "~" H 970 1640 50  0001 C CNN
+F 2 "Resistor_SMD:R_0603_1608Metric_Pad1.05x0.95mm_HandSolder" H 970 1640 50  0001 C CNN
+F 3 "https://lcsc.com/product-detail/Chip-Resistor-Surface-Mount_YAGEO-RC0603JR-071K1L_C246023.html" H 970 1640 50  0001 C CNN
+F 4 "RC0603JR-071K1L" H 970 1640 50  0001 C CNN "manf#"
 	1    970  1640
 	1    0    0    -1
@@
 F 0 "R1" V 1426 3000 50  0000 C CNN
 F 1 "1K" V 1335 3000 50  0000 C CNN
-F 2 "" H 1230 3000 50  0001 C CNN
-F 3 "~" H 1230 3000 50  0001 C CNN
+F 2 "Resistor_SMD:R_0603_1608Metric_Pad1.05x0.95mm_HandSolder" H 1230 3000 50  0001 C CNN
+F 3 "https://lcsc.com/product-detail/Chip-Resistor-Surface-Mount_YAGEO-RC0603JR-071K1L_C246023.html" H 1230 3000 50  0001 C CNN
+F 4 "RC0603JR-071K1L" H 1230 3000 50  0001 C CNN "manf#"
 	1    1230 3000
 	0    -1   -1   0
@@
 F 0 "R5" H 2379 2826 50  0000 L CNN
 F 1 "1K" H 2379 2735 50  0000 L CNN
-F 2 "" H 2320 2780 50  0001 C CNN
-F 3 "~" H 2320 2780 50  0001 C CNN
+F 2 "Resistor_SMD:R_0603_1608Metric_Pad1.05x0.95mm_HandSolder" H 2320 2780 50  0001 C CNN
+F 3 "https://lcsc.com/product-detail/Chip-Resistor-Surface-Mount_YAGEO-RC0603JR-071K1L_C246023.html" H 2320 2780 50  0001 C CNN
+F 4 "RC0603JR-071K1L" H 2320 2780 50  0001 C CNN "manf#"
 	1    2320 2780
 	1    0    0    -1
@@
 P 4760 1640
 F 0 "C1" H 4852 1686 50  0000 L CNN
-F 1 "C_Small" H 4852 1595 50  0000 L CNN
-F 2 "" H 4760 1640 50  0001 C CNN
-F 3 "~" H 4760 1640 50  0001 C CNN
+F 1 "0.1uF" H 4852 1595 50  0000 L CNN
+F 2 "Capacitor_SMD:C_0603_1608Metric" H 4760 1640 50  0001 C CNN
+F 3 "https://lcsc.com/product-detail/Multilayer-Ceramic-Capacitors-MLCC-SMD-SMT_Walsin-Tech-Corp-0603F104Z160CT_C387984.html" H 4760 1640 50  0001 C CNN
+F 4 "0603F104Z160CT" H 4760 1640 50  0001 C CNN "manf#"
 	1    4760 1640
 	1    0    0    -1
@@
 F 0 "R9" H 5281 1594 50  0000 R CNN
 F 1 "4.7K" H 5281 1685 50  0000 R CNN
-F 2 "" H 5340 1640 50  0001 C CNN
-F 3 "~" H 5340 1640 50  0001 C CNN
+F 2 "Resistor_SMD:R_0805_2012Metric_Pad1.15x1.40mm_HandSolder" H 5340 1640 50  0001 C CNN
+F 3 "https://lcsc.com/product-detail/Chip-Resistor-Surface-Mount_FH-Guangdong-Fenghua-Advanced-Tech-RS-05K472JT_C115310.html" H 5340 1640 50  0001 C CNN
+F 4 "RS-05K472JT" H 5340 1640 50  0001 C CNN "manf#"
 	1    5340 1640
 	-1   0    0    1
@@
 F 0 "R11" H 5761 1594 50  0000 R CNN
 F 1 "4.7K" H 5761 1685 50  0000 R CNN
-F 2 "" H 5820 1640 50  0001 C CNN
-F 3 "~" H 5820 1640 50  0001 C CNN
+F 2 "Resistor_SMD:R_0805_2012Metric_Pad1.15x1.40mm_HandSolder" H 5820 1640 50  0001 C CNN
+F 3 "https://lcsc.com/product-detail/Chip-Resistor-Surface-Mount_FH-Guangdong-Fenghua-Advanced-Tech-RS-05K472JT_C115310.html" H 5820 1640 50  0001 C CNN
+F 4 "RS-05K472JT" H 5820 1640 50  0001 C CNN "manf#"
 	1    5820 1640
 	-1   0    0    1
@@
 F 0 "R8" H 4991 2654 50  0000 R CNN
 F 1 "120R" H 4991 2745 50  0000 R CNN
-F 2 "" H 5050 2700 50  0001 C CNN
-F 3 "~" H 5050 2700 50  0001 C CNN
+F 2 "Resistor_SMD:R_0603_1608Metric_Pad1.05x0.95mm_HandSolder" H 5050 2700 50  0001 C CNN
+F 3 "https://lcsc.com/product-detail/Chip-Resistor-Surface-Mount_UNI-ROYAL-Uniroyal-Elec-0603SAJ0121T5E_C303866.html" H 5050 2700 50  0001 C CNN
+F 4 "0603SAJ0121T5E" H 5050 2700 50  0001 C CNN "manf#"
 	1    5050 2700
 	-1   0    0    1
@@
 F 0 "J1" H 7490 2032 50  0000 L CNN
 F 1 "Screw_Terminal_01x02" H 7490 1941 50  0000 L CNN
-F 2 "" H 7410 2040 50  0001 C CNN
+F 2 "TerminalBlock:TerminalBlock_Altech_AK300-2_P5.00mm" H 7410 2040 50  0001 C CNN
 F 3 "~" H 7410 2040 50  0001 C CNN
 	1    7410 2040
@@
 Wire Notes Line
 	470  3750 11180 3750
+$Comp
+L Connector_Generic:Conn_01x16 J1
+U 1 1 5D375C76
+P 9100 1700
+F 0 "J1" H 9019 675 50  0000 C CNN
+F 1 "feather long" H 9019 766 50  0000 C CNN
+F 2 "TerminalBlock:TerminalBlock_Altech_AK300-2_P5.00mm" H 9100 1700 50  0001 C CNN
+F 3 "~" H 9100 1700 50  0001 C CNN
+	1    9100 1700
+	1    0    0    1
+$EndComp
+$Comp
+L Connector_Generic:Conn_01x12 J2
+U 1 1 5D375CC4
+P 9500 1900
+F 0 "J2" H 9420 1075 50  0000 C CNN
+F 1 "feather short" H 9420 1166 50  0000 C CNN
+F 2 "Connector_PinHeader_2.54mm:PinHeader_1x12_P2.54mm_Vertical" H 9500 1900 50  0001 C CNN
+F 3 "" H 9500 1900 50  0001 C CNN
+	1    9500 1900
+	-1   0    0    1
+$EndComp
+Text Label 8700 900  0    50   ~ 0
+~RST
+Text Label 8700 1100 0    50   ~ 0
+AREF
+Text Label 8700 1300 0    50   ~ 0
+A0
+Text Label 8700 1400 0    50   ~ 0
+A1
+Text Label 8700 1500 0    50   ~ 0
+A2
+Text Label 8700 1600 0    50   ~ 0
+A3
+Text Label 8700 1700 0    50   ~ 0
+A4
+Text Label 8700 1800 0    50   ~ 0
+A5
+Text Label 8700 1900 0    50   ~ 0
+SCK
+Text Label 8700 2000 0    50   ~ 0
+MOSI
+Text Label 8700 2100 0    50   ~ 0
+MISO
+Text Label 8700 2200 0    50   ~ 0
+RX
+Text Label 8700 2300 0    50   ~ 0
+TX
+Text Label 8700 2400 0    50   ~ 0
+FREE
+Text Label 9950 1300 2    50   ~ 0
+VBAT
+Text Label 9950 1400 2    50   ~ 0
+EN
+Text Label 9950 1500 2    50   ~ 0
+VUSB
+Text Label 9950 1600 2    50   ~ 0
+D6
+Text Label 9950 1700 2    50   ~ 0
+D5
+Text Label 9950 1800 2    50   ~ 0
+D4
+Text Label 9950 1900 2    50   ~ 0
+D3
+Text Label 9950 2000 2    50   ~ 0
+D2
+Text Label 9950 2100 2    50   ~ 0
+D1
+Text Label 9950 2200 2    50   ~ 0
+D0
+Text Label 9950 2300 2    50   ~ 0
+SCL
+Text Label 9950 2400 2    50   ~ 0
+SDA
+Wire Wire Line
+	8700 900  8900 900
+Wire Wire Line
+	8700 1100 8900 1100
+Wire Wire Line
+	8700 1300 8900 1300
+Wire Wire Line
+	8700 1400 8900 1400
+Wire Wire Line
+	8700 1500 8900 1500
+Wire Wire Line
+	8700 1600 8900 1600
+Wire Wire Line
+	8700 1700 8900 1700
+Wire Wire Line
+	8700 1800 8900 1800
+Wire Wire Line
+	8700 1900 8900 1900
+Wire Wire Line
+	8700 2000 8900 2000
+Wire Wire Line
+	8700 2100 8900 2100
+Wire Wire Line
+	8700 2200 8900 2200
+Wire Wire Line
+	8700 2300 8900 2300
+Wire Wire Line
+	8700 2400 8900 2400
+Wire Wire Line
+	9700 1300 9950 1300
+Wire Wire Line
+	9700 1400 9950 1400
+Wire Wire Line
+	9700 1500 9950 1500
+Wire Wire Line
+	9700 1600 9950 1600
+Wire Wire Line
+	9700 1700 9950 1700
+Wire Wire Line
+	9700 1800 9950 1800
+Wire Wire Line
+	9700 1900 9950 1900
+Wire Wire Line
+	9700 2000 9950 2000
+Wire Wire Line
+	9700 2100 9950 2100
+Wire Wire Line
+	9700 2200 9950 2200
+Wire Wire Line
+	9700 2300 9950 2300
+Wire Wire Line
+	9700 2400 9950 2400
+$Comp
+L power:+3.3V #PWR0101
+U 1 1 5D37877D
+P 8550 900
+F 0 "#PWR0101" H 8550 750 50  0001 C CNN
+F 1 "+3.3V" H 8565 1073 50  0000 C CNN
+F 2 "" H 8550 900 50  0001 C CNN
+F 3 "" H 8550 900 50  0001 C CNN
+	1    8550 900
+	1    0    0    -1
+$EndComp
+$Comp
+L power:GND #PWR0102
+U 1 1 5D3787E4
+P 8550 1300
+F 0 "#PWR0102" H 8550 1050 50  0001 C CNN
+F 1 "GND" H 8555 1127 50  0000 C CNN
+F 2 "" H 8550 1300 50  0001 C CNN
+F 3 "" H 8550 1300 50  0001 C CNN
+	1    8550 1300
+	1    0    0    -1
+$EndComp
+Wire Wire Line
+	8550 900  8550 1000
+Wire Wire Line
+	8550 1000 8900 1000
+Wire Wire Line
+	8550 1300 8550 1200
+Wire Wire Line
+	8550 1200 8900 1200
+Wire Notes Line
+	8350 500  8350 3750
 $EndSCHEMATC

Commit message: Add_netlist
Parts:
- renumbered J1 to J3, R2 to R1, R9 to R2, R11 to R3, R6 to R4, R7 to R5, R8 to R6, R5 to R7, R1 to R8, U2 to U1, U3 to U2, U1 to U3
Changed lines of the file:
@@
 $EndDescr
 $Comp
-L Interface_UART:MAX487E U3
+L Interface_UART:MAX487E U2
 U 1 1 5F9AD072
 P 4190 2670
-F 0 "U3" H 3900 3270 50  0000 C CNN
+F 0 "U2" H 3900 3270 50  0000 C CNN
 F 1 "MAX13487E" H 3920 3180 50  0000 C CNN
 F 2 "Package_SO:SOIC-8_3.9x4.9mm_P1.27mm" H 4190 1970 50  0001 C CNN
@@
 $EndComp
 $Comp
-L RS485_Modbus_Wing-rescue:VOS617A-Isolatorr U1
+L RS485_Modbus_Wing-rescue:VOS617A-Isolatorr U3
 U 1 1 5F9C2337
 P 1950 2900
-F 0 "U1" H 1701 2483 50  0000 C CNN
+F 0 "U3" H 1701 2483 50  0000 C CNN
 F 1 "VOS617A" H 1850 2934 50  0000 C CNN
 F 2 "Package_SO:SO-4_4.4x2.3mm_P1.27mm" H 1950 2900 50  0001 C CNN
@@
 $EndComp
 $Comp
-L RS485_Modbus_Wing-rescue:VOS617A-Isolatorr U2
+L RS485_Modbus_Wing-rescue:VOS617A-Isolatorr U1
 U 1 1 5F9C0BC7
 P 1350 1770
-F 0 "U2" H 1366 1785 50  0000 C CNN
+F 0 "U1" H 1366 1785 50  0000 C CNN
 F 1 "VOS617A" H 1166 1349 50  0000 C CNN
 F 2 "Package_SO:SO-4_4.4x2.3mm_P1.27mm" H 1350 1770 50  0001 C CNN
@@
 $EndComp
 $Comp
-L power:GND #PWR04
+L power:GND #PWR0101
 U 1 1 5F9D5FDD
 P 2250 3270
-F 0 "#PWR04" H 2250 3020 50  0001 C CNN
+F 0 "#PWR0101" H 2250 3020 50  0001 C CNN
 F 1 "GND" H 2255 3097 50  0000 C CNN
 F 2 "" H 2250 3270 50  0001 C CNN
@@
 	2250 3200 2250 3270
 $Comp
-L Device:R_Small R7
+L Device:R_Small R5
 U 1 1 5F9D8466
 P 3340 2160
-F 0 "R7" H 3281 2114 50  0000 R CNN
+F 0 "R5" H 3281 2114 50  0000 R CNN
 F 1 "4.7K" H 3281 2205 50  0000 R CNN
 F 2 "Resistor_SMD:R_0805_2012Metric_Pad1.15x1.40mm_HandSolder" H 3340 2160 50  0001 C CNN
@@
 	3340 2670 3340 2260
 $Comp
-L power:VBUS #PWR07
+L power:VBUS #PWR0102
 U 1 1 5F9D96A3
 P 3340 1800
-F 0 "#PWR07" H 3340 1650 50  0001 C CNN
+F 0 "#PWR0102" H 3340 1650 50  0001 C CNN
 F 1 "VBUS" H 3355 1973 50  0000 C CNN
 F 2 "" H 3340 1800 50  0001 C CNN
@@
 	3790 2570 3700 2570
 $Comp
-L power:VBUS #PWR06
+L power:VBUS #PWR0103
 U 1 1 5F9DBA8D
 P 1870 1530
-F 0 "#PWR06" H 1870 1380 50  0001 C CNN
+F 0 "#PWR0103" H 1870 1380 50  0001 C CNN
 F 1 "VBUS" H 1885 1703 50  0000 C CNN
 F 2 "" H 1870 1530 50  0001 C CNN
@@
 $EndComp
 $Comp
-L Device:R_Small R6
+L Device:R_Small R4
 U 1 1 5F9DBA98
 P 1870 1750
-F 0 "R6" H 1811 1704 50  0000 R CNN
+F 0 "R4" H 1811 1704 50  0000 R CNN
 F 1 "1K" H 1811 1795 50  0000 R CNN
 F 2 "Resistor_SMD:R_0603_1608Metric_Pad1.05x0.95mm_HandSolder" H 1870 1750 50  0001 C CNN
@@
 Connection ~ 970  1870
 $Comp
-L Device:R_Small R2
+L Device:R_Small R1
 U 1 1 5F9E2582
 P 970 1640
-F 0 "R2" H 820 1670 50  0000 L CNN
+F 0 "R1" H 820 1670 50  0000 L CNN
 F 1 "1K" H 810 1600 50  0000 L CNN
 F 2 "Resistor_SMD:R_0603_1608Metric_Pad1.05x0.95mm_HandSolder" H 970 1640 50  0001 C CNN
@@
 	970  1540 970  1490
 $Comp
-L power:+3.3V #PWR02
+L power:+3.3V #PWR0104
 U 1 1 5F9E37F5
 P 970 1490
-F 0 "#PWR02" H 970 1340 50  0001 C CNN
+F 0 "#PWR0104" H 970 1340 50  0001 C CNN
 F 1 "+3.3V" H 985 1663 50  0000 C CNN
 F 2 "" H 970 1490 50  0001 C CNN
@@
 $EndComp
 $Comp
-L power:+3.3V #PWR01
+L power:+3.3V #PWR0105
 U 1 1 5F9E483C
 P 860 2930
-F 0 "#PWR01" H 860 2780 50  0001 C CNN
+F 0 "#PWR0105" H 860 2780 50  0001 C CNN
 F 1 "+3.3V" H 875 3103 50  0000 C CNN
 F 2 "" H 860 2930 50  0001 C CNN
@@
 $EndComp
 $Comp
-L Device:R_Small R1
+L Device:R_Small R8
 U 1 1 5F9E5C52
 P 1230 3000
-F 0 "R1" V 1426 3000 50  0000 C CNN
+F 0 "R8" V 1426 3000 50  0000 C CNN
 F 1 "1K" V 1335 3000 50  0000 C CNN
 F 2 "Resistor_SMD:R_0603_1608Metric_Pad1.05x0.95mm_HandSolder" H 1230 3000 50  0001 C CNN
@@
 D1TX
 $Comp
-L power:GND #PWR03
+L power:GND #PWR0106
 U 1 1 5F9E7A11
 P 1110 2120
-F 0 "#PWR03" H 1110 1870 50  0001 C CNN
+F 0 "#PWR0106" H 1110 1870 50  0001 C CNN
 F 1 "GND" H 1115 1947 50  0000 C CNN
 F 2 "" H 1110 2120 50  0001 C CNN
@@
 	1110 2070 1110 2120
 $Comp
-L Device:R_Small R5
+L Device:R_Small R7
 U 1 1 5F9EA1EE
 P 2320 2780
-F 0 "R5" H 2379 2826 50  0000 L CNN
+F 0 "R7" H 2379 2826 50  0000 L CNN
 F 1 "1K" H 2379 2735 50  0000 L CNN
 F 2 "Resistor_SMD:R_0603_1608Metric_Pad1.05x0.95mm_HandSolder" H 2320 2780 50  0001 C CNN
@@
 	2320 2880 2320 3000
 $Comp
-L power:VBUS #PWR05
+L power:VBUS #PWR0107
 U 1 1 5F9EBFD8
 P 2320 2610
-F 0 "#PWR05" H 2320 2460 50  0001 C CNN
+F 0 "#PWR0107" H 2320 2460 50  0001 C CNN
 F 1 "VBUS" H 2335 2783 50  0000 C CNN
 F 2 "" H 2320 2610 50  0001 C CNN
@@
 $EndComp
 $Comp
-L power:GND #PWR09
+L power:GND #PWR0108
 U 1 1 5F9ED13F
 P 4190 3400
-F 0 "#PWR09" H 4190 3150 50  0001 C CNN
+F 0 "#PWR0108" H 4190 3150 50  0001 C CNN
 F 1 "GND" H 4195 3227 50  0000 C CNN
 F 2 "" H 4190 3400 50  0001 C CNN
@@
 	4190 3270 4190 3400
 $Comp
-L power:VBUS #PWR08
+L power:VBUS #PWR0109
 U 1 1 5F9EE32B
 P 4190 1980
-F 0 "#PWR08" H 4190 1830 50  0001 C CNN
+F 0 "#PWR0109" H 4190 1830 50  0001 C CNN
 F 1 "VBUS" H 4205 2153 50  0000 C CNN
 F 2 "" H 4190 1980 50  0001 C CNN
@@
 	4190 2170 4190 1980
 $Comp
-L power:VBUS #PWR010
+L power:VBUS #PWR0110
 U 1 1 5F9F0C0C
 P 4760 1470
-F 0 "#PWR010" H 4760 1320 50  0001 C CNN
+F 0 "#PWR0110" H 4760 1320 50  0001 C CNN
 F 1 "VBUS" H 4775 1643 50  0000 C CNN
 F 2 "" H 4760 1470 50  0001 C CNN
@@
 	4760 1470 4760 1540
 $Comp
-L power:GND #PWR011
+L power:GND #PWR0111
 U 1 1 5F9F297E
 P 4760 1810
-F 0 "#PWR011" H 4760 1560 50  0001 C CNN
+F 0 "#PWR0111" H 4760 1560 50  0001 C CNN
 F 1 "GND" H 4765 1637 50  0000 C CNN
 F 2 "" H 4760 1810 50  0001 C CNN
@@
 	4760 1810 4760 1740
 $Comp
-L Device:R_Small R9
+L Device:R_Small R2
 U 1 1 5F9F467C
 P 5340 1640
-F 0 "R9" H 5281 1594 50  0000 R CNN
+F 0 "R2" H 5281 1594 50  0000 R CNN
 F 1 "4.7K" H 5281 1685 50  0000 R CNN
 F 2 "Resistor_SMD:R_0805_2012Metric_Pad1.15x1.40mm_HandSolder" H 5340 1640 50  0001 C CNN
@@
 $EndComp
 $Comp
-L power:VBUS #PWR012
+L power:VBUS #PWR0112
 U 1 1 5F9F4B91
 P 5340 1460
-F 0 "#PWR012" H 5340 1310 50  0001 C CNN
+F 0 "#PWR0112" H 5340 1310 50  0001 C CNN
 F 1 "VBUS" H 5355 1633 50  0000 C CNN
 F 2 "" H 5340 1460 50  0001 C CNN
@@
 	5340 1740 5340 1910
 $Comp
-L Device:R_Small R11
+L Device:R_Small R3
 U 1 1 5F9F94E0
 P 5820 1640
-F 0 "R11" H 5761 1594 50  0000 R CNN
+F 0 "R3" H 5761 1594 50  0000 R CNN
 F 1 "4.7K" H 5761 1685 50  0000 R CNN
 F 2 "Resistor_SMD:R_0805_2012Metric_Pad1.15x1.40mm_HandSolder" H 5820 1640 50  0001 C CNN
@@
 	5820 1540 5820 1460
 $Comp
-L power:GND #PWR013
+L power:GND #PWR0113
 U 1 1 5F9FAABB
 P 5820 1850
-F 0 "#PWR013" H 5820 1600 50  0001 C CNN
+F 0 "#PWR0113" H 5820 1600 50  0001 C CNN
 F 1 "GND" H 5825 1677 50  0000 C CNN
 F 2 "" H 5820 1850 50  0001 C CNN
@@
 B
 $Comp
-L Device:R_Small R8
+L Device:R_Small R6
 U 1 1 5F9FCB14
 P 5050 2700
-F 0 "R8" H 4991 2654 50  0000 R CNN
+F 0 "R6" H 4991 2654 50  0000 R CNN
 F 1 "120R" H 4991 2745 50  0000 R CNN
 F 2 "Resistor_SMD:R_0603_1608Metric_Pad1.05x0.95mm_HandSolder" H 5050 2700 50  0001 C CNN
@@
 RS485A
 $Comp
-L Connector:Screw_Terminal_01x02 J1
+L Connector:Screw_Terminal_01x02 J3
 U 1 1 5FA0A2EE
 P 7410 2040
-F 0 "J1" H 7490 2032 50  0000 L CNN
+F 0 "J3" H 7490 2032 50  0000 L CNN
 F 1 "Screw_Terminal_01x02" H 7490 1941 50  0000 L CNN
 F 2 "TerminalBlock:TerminalBlock_Altech_AK300-2_P5.00mm" H 7410 2040 50  0001 C CNN
@@
 	9700 2400 9950 2400
 $Comp
-L power:+3.3V #PWR0101
+L power:+3.3V #PWR0114
 U 1 1 5D37877D
 P 8550 900
-F 0 "#PWR0101" H 8550 750 50  0001 C CNN
+F 0 "#PWR0114" H 8550 750 50  0001 C CNN
 F 1 "+3.3V" H 8565 1073 50  0000 C CNN
 F 2 "" H 8550 900 50  0001 C CNN
@@
 $EndComp
 $Comp
-L power:GND #PWR0102
+L power:GND #PWR0115
 U 1 1 5D3787E4
 P 8550 1300
-F 0 "#PWR0102" H 8550 1050 50  0001 C CNN
+F 0 "#PWR0115" H 8550 1050 50  0001 C CNN
 F 1 "GND" H 8555 1127 50  0000 C CNN
 F 2 "" H 8550 1300 50  0001 C CNN

Commit message: Fist_PCB
Connections:
- net D0 is gone; now on net D0RX: J2.3 (Pin_3)
- net D1 is gone; now on net D1TX: J2.4 (Pin_4)
- net VUSB is gone; now on net VBUS: J2.10 (Pin_10)
- net DI: now also R7.2, U3.4
Other:
- note added: "INPUTS\n"
- note added: "OUTPUTS\n"
- note added: "PINS"
- note added: "RS485"
Changed lines of the file:
@@
 encoding utf-8
 Sheet 1 1
-Title ""
-Date ""
-Rev ""
-Comp ""
+Title "RS485"
+Date "2020-11-03"
+Rev "1.0"
+Comp "Electronic Cats"
 Comment1 ""
 Comment2 ""
@@
 EN
 Text Label 9950 1500 2    50   ~ 0
-VUSB
+VBUS
 Text Label 9950 1600 2    50   ~ 0
 D6
@@
 D2
 Text Label 9950 2100 2    50   ~ 0
-D1
+D1TX
 Text Label 9950 2200 2    50   ~ 0
-D0
+D0RX
 Text Label 9950 2300 2    50   ~ 0
 SCL
@@
 Wire Notes Line
 	8350 500  8350 3750
+Text Label 2490 3000 0    50   ~ 0
+DI
+Wire Wire Line
+	2320 3000 2490 3000
+Connection ~ 2320 3000
+Text Notes 530  620  0    50   ~ 0
+INPUTS\n
+Text Notes 2940 580  0    50   ~ 0
+RS485
+Text Notes 6780 670  0    50   ~ 0
+OUTPUTS\n
+Text Notes 8480 590  0    50   ~ 0
+PINS
 $EndSCHEMATC

Commit message: Add_Logo
Parts:
- J3: footprint TerminalBlock:TerminalBlock_Altech_AK300-2_P5.00mm -> TerminalBlock:TerminalBlock_bornier-2_P5.08mm
Changed lines of the file:
@@
 F 0 "J3" H 7490 2032 50  0000 L CNN
 F 1 "Screw_Terminal_01x02" H 7490 1941 50  0000 L CNN
-F 2 "TerminalBlock:TerminalBlock_Altech_AK300-2_P5.00mm" H 7410 2040 50  0001 C CNN
+F 2 "TerminalBlock:TerminalBlock_bornier-2_P5.08mm" H 7410 2040 50  0001 C CNN
 F 3 "~" H 7410 2040 50  0001 C CNN
 	1    7410 2040

Commit message: Last_Revision
Connections:
- net RX: now also R1.2, U1.4
- net TX: now also U3.2
- removed net D0RX: J2.3 (Pin_3), R1.2, U1.4
- net D1TX renamed D1
- net D1: no longer U3.2
- new net D0: J2.3 (Pin_3)
Changed lines of the file:
@@
 Wire Wire Line
 	1870 1650 1870 1530
-Text Label 870  1870 2    50   ~ 0
-D0RX
 Wire Wire Line
 	870  1870 970  1870
@@
 Wire Wire Line
 	860  3000 860  2930
-Text Label 1440 3200 2    50   ~ 0
-D1TX
 $Comp
 L power:GND #PWR0106
@@
 Text Label 9950 2000 2    50   ~ 0
 D2
-Text Label 9950 2100 2    50   ~ 0
-D1TX
-Text Label 9950 2200 2    50   ~ 0
-D0RX
 Text Label 9950 2300 2    50   ~ 0
 SCL
@@
 Text Notes 8480 590  0    50   ~ 0
 PINS
+Text Label 9950 2100 2    50   ~ 0
+D1
+Text Label 9950 2200 2    50   ~ 0
+D0
+Text Label 1440 3200 2    50   ~ 0
+TX
+Text Label 870  1870 2    50   ~ 0
+RX
 $EndSCHEMATC

Commit message: change_pin
Connections:
- net D0 is gone; now on net D5: J2.3 (Pin_3)
- net D1 is gone; now on net D6: J2.4 (Pin_4)
- net D5: no longer J2.8 (Pin_8)
- net D6: no longer J2.9 (Pin_9)
- net D2 renamed D9
- net D3 renamed D10
- net D4 renamed D11
- new net D12: J2.8 (Pin_8)
- new net D13: J2.9 (Pin_9)
Changed lines of the file:
@@
 VBUS
 Text Label 9950 1600 2    50   ~ 0
-D6
+D13
 Text Label 9950 1700 2    50   ~ 0
-D5
+D12
 Text Label 9950 1800 2    50   ~ 0
-D4
+D11
 Text Label 9950 1900 2    50   ~ 0
-D3
+D10
 Text Label 9950 2000 2    50   ~ 0
-D2
+D9
 Text Label 9950 2300 2    50   ~ 0
 SCL
@@
 PINS
 Text Label 9950 2100 2    50   ~ 0
-D1
+D6
 Text Label 9950 2200 2    50   ~ 0
-D0
+D5
 Text Label 1440 3200 2    50   ~ 0
 TX
