File: RS485_Modbus_Wing.sch (KiCad schematic (older format))
At the start: 15 parts, among them J1 feather long, J2 feather short, J3 Screw_Terminal_01x02, U1 VOS617A, U2 MAX13487E, U3 VOS617A

Commit message: ChangeRS
Parts:
- removed R8: 1K, Resistor_SMD:R_0603_1608Metric_Pad1.05x0.95mm_HandSolder, symbol Device:R_Small
- removed U1, U3: VOS617A, Package_SO:SO-4_4.4x2.3mm_P1.27mm, symbol RS485_Modbus_Wing-rescue:VOS617A-Isolatorr
- removed U2: MAX13487E, Package_SO:SOIC-8_3.9x4.9mm_P1.27mm, symbol Interface_UART:MAX487E
- added C2: 0.1uF, Capacitor_SMD:C_0603_1608Metric_Pad1.05x0.95mm_HandSolder, symbol Device:C_Small
- added U1: SP3485EN, Package_SO:SOIC-8_3.9x4.9mm_P1.27mm, symbol Interface_UART:SP3485EN
- C1: value 0.1uF -> 10uF; footprint Capacitor_SMD:C_0603_1608Metric -> Capacitor_SMD:C_0603_1608Metric_Pad1.05x0.95mm_HandSolder; manf# 0603F104Z160CT -> (none)
- R1, R4: value 1K -> 10K; manf# RC0603JR-071K1L -> (none)
- R2, R3: value 4.7K -> 10K; footprint Resistor_SMD:R_0805_2012Metric_Pad1.15x1.40mm_HandSolder -> Resistor_SMD:R_0603_1608Metric_Pad1.05x0.95mm_HandSolder; manf# RS-05K472JT -> (none)
- R5: value 4.7K -> 20K; footprint Resistor_SMD:R_0805_2012Metric_Pad1.15x1.40mm_HandSolder -> Resistor_SMD:R_0603_1608Metric_Pad1.05x0.95mm_HandSolder; manf# RS-05K472JT -> (none)
- R6: value 120R -> 120; manf# 0603SAJ0121T5E -> (none)
- R7: value 1K -> 20K; manf# RC0603JR-071K1L -> (none)
Connections:
- net D12 is gone; now on net DI: J2.8 (Pin_8)
- net D9 is gone; now on net RO: J2.5 (Pin_5)
- net +3V3: now also C1.1, R2.1, R3.1, R4.1, R7.2, C2.1, U1.8 (VCC)
- net DI: now also R4.2, U1.4 (DI); no longer R7.2
- net GND: now also R5.1, C2.2, U1.5 (GND); no longer R3.1
- net RO: now also R1.2, U1.1 (RO)
- net RX: no longer R1.2
- net VBUS: no longer C1.1, R2.2, R4.2, R5.2, R7.1
- removed net A: J3.2 (Pin_2), R2.1, R6.1
- removed net B: J3.1 (Pin_1), R3.2, R6.2
- net D10 renamed RE
- net RE: now also R2.2, U1.2 (~RE~)
- net D11 renamed DE
- net DE: now also R3.2, U1.3 (DE)
- new net RS485A: J3.2 (Pin_2), R6.2, R7.1, U1.6 (A)
- new net RS485B: J3.1 (Pin_1), R5.2, R6.1, U1.7 (B)
Other:
- note removed: "INPUTS\n"
