File: Hw/RS485_Modbus_Wing.sch (KiCad schematic (older format))
At the start: 13 parts, among them J1 feather long, J2 feather short, J3 Screw_Terminal_01x02, U1 SP3485EN

Commit message: fix layout
Connections:
- net DE: now also J2.6 (Pin_6); no longer J2.7 (Pin_7)
- net RE: now also J2.7 (Pin_7); no longer J2.6 (Pin_6)
Changed lines of the file:
@@
 Text Label 9950 1600 2    50   ~ 0
 D13
-Text Label 9950 1800 2    50   ~ 0
+Text Label 9950 1900 2    50   ~ 0
 DE
 Wire Wire Line
@@
 Wire Wire Line
 	9700 1900 9950 1900
-Text Label 9950 1900 2    50   ~ 0
+Text Label 9950 1800 2    50   ~ 0
 RE
 Text Label 8700 2300 0    50   ~ 0
