File: Hw/RS485_Modbus_Wing.kicad_pcb (KiCad board)
At the start: 2 copper layers, 50.8 x 22.9 mm, 20 parts, among them J1 feather long, J2 feather short, J3 Screw_Terminal_01x02, U1 SP3485EN

Commit message: fix layout
Parts:
- moved R7 15.2 mm to (163.8, 89.0), turned to 270 degrees
- moved R6 12.9 mm to (163.7, 85.6), turned to 270 degrees
- moved R5 12.1 mm to (163.7, 82.3), turned to 270 degrees
- moved C2 11.6 mm to (157.9, 82.1), turned to 180 degrees
- moved C1 9.35 mm to (161.8, 82.2), turned to 90 degrees
- moved R2 8.28 mm to (149.0, 82.7)
- moved R1 6.57 mm to (150.5, 82.7), turned to 270 degrees
- moved U1 4.34 mm to (155.9, 85.5), turned to 0 degrees
- moved R3 2.38 mm to (147.6, 82.7), turned to 270 degrees
- moved R4 2.33 mm to (146.1, 82.7), turned to 270 degrees
Connections:
- J2 pad 6: /RE -> /DE
- J2 pad 7: /DE -> /RE
Routing:
- net /RS485B: track 31.9 -> 13.5 mm
- net +3V3: track 52.7 -> 70.7 mm, vias 1 -> 2
- net /RS485A: track 29.6 -> 13.6 mm
- net GND: track 14.3 -> 29.9 mm, vias 4 -> 6
- net /DE: track 12.0 -> 21.4 mm
- net /TX: track 36.2 -> 30.4 mm
- net /RE: track 14.5 -> 18.9 mm
- net /RX: track 22.2 -> 25.5 mm, vias 1 -> 2

Commit message: add solder mask clearence
Other:
- rule pad_to_mask_clearance: 0.051 -> 0
