File: Hw/RS485_Modbus_Wing.kicad_pcb (KiCad board)
At the start: 2 copper layers, 50.8 x 22.9 mm, 20 parts, among them J1 feather long, J2 feather short, J3 Screw_Terminal_01x02, U1 SP3485EN

Commit message: Update_Kicad_6
Connections:
- net /~RST renamed /~{RST}
Other:
- net class Default removed
- net class Source removed
- board text added: "~{RST}"
- board text removed: "~RST"
