File: Hw/RS485_Modbus_Wing.kicad_sch (KiCad schematic)
At the start: 13 parts, among them J1 feather long, J2 feather short, J3 Screw_Terminal_01x02, U1 SP3485EN

Commit message: BOM update and generated
Parts:
- C1: value 10uF -> (none); footprint Capacitor_SMD:C_0603_1608Metric_Pad1.05x0.95mm_HandSolder -> (none); LCSC# (none) -> C326057; Proveedor (none) -> LCSC
- C2: value 0.1uF -> (none); footprint Capacitor_SMD:C_0603_1608Metric_Pad1.05x0.95mm_HandSolder -> (none); Proveedor (none) -> MOUSER
- J1: value feather long -> (none); footprint TerminalBlock:TerminalBlock_Altech_AK300-2_P5.00mm -> (none)
- J2: value feather short -> (none); footprint Connector_PinHeader_2.54mm:PinHeader_1x12_P2.54mm_Vertical -> (none)
- J3: value Screw_Terminal_01x02 -> (none); footprint TerminalBlock:TerminalBlock_bornier-2_P5.08mm -> (none); LCSC# (none) -> C8465; Proveedor (none) -> LCSC
- R1, R2, R3, R4: value 10K -> (none); footprint Resistor_SMD:R_0603_1608Metric_Pad1.05x0.95mm_HandSolder -> (none); Proveedor (none) -> MOUSER
- R5, R7: value 20K -> (none); footprint Resistor_SMD:R_0603_1608Metric_Pad1.05x0.95mm_HandSolder -> (none); LCSC# (none) -> C25586; Proveedor (none) -> LCSC
- R6: value 120 -> (none); footprint Resistor_SMD:R_0603_1608Metric_Pad1.05x0.95mm_HandSolder -> (none); LCSC# (none) -> C103256; Proveedor (none) -> LCSC
- U1: value SP3485EN -> (none); footprint Package_SO:SOIC-8_3.9x4.9mm_P1.27mm -> (none); Proveedor (none) -> MOUSER; manf# SP3485CN -> SP3485EN-L/TR
